File: microgame2.kicad_sch (KiCad schematic)
At the start: 17 parts, among them SW9 SW_SPST, U1 ESP32-PICO-D4

Commit message: reverting
Other:
- removed sheet Power2

Commit message: updating main sch
Other:
- added sheet Power2 (power.kicad_sch)
