File: microgame2.kicad_sch (KiCad schematic)
At the start: 17 parts, among them SW9 SW_SPST, U1 ESP32-PICO-D4

Commit message: adding sheet
Other:
- added sheet Power2 (power.kicad_sch)
Changed lines of the file:
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@@
+    )
+  )
+  (sheet (at 67.31 31.0384) (size 40.64 6.35) (fields_autoplaced)
+    (stroke (width 0) (type solid))
+    (fill (color 0 0 0 0.0000))
+    (property "Sheetname" "Power2" (at 67.31 19.6084 0)
+      (effects (font (size 1.27 1.27)) (justify left bottom))
+    )
+    (property "Sheetfile" "power.kicad_sch" (at 67.31 27.2546 0)
+      (effects (font (size 1.27 1.27)) (justify left top))
+    )
+    (pin "Foo" input (at 90.17 31.75 90)
+      (effects (font (size 1.27 1.27)) (justify right))
+    )
+    (instances
+      (project "microgame2"
+        (path "/ebfd9da1-8e1c-4303-a1cc-72875a794180" (page "7"))
+      )
     )
   )

Commit message: adding more sheets
Other:
- added sheet Power3 (power.kicad_sch)
- added sheet Power4 (power.kicad_sch)
Changed lines of the file:
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@@
+    )
+  )
+  (sheet (at 67.31 42.4684 0) (size 40.64 6.35) (fields_autoplaced)
+    (stroke (width 0) (type solid))
+    (fill (color 0 0 0 0.0000))
+    (property "Sheetname" "Power3" (at 67.31 19.6084 0)
+      (effects (font (size 1.27 1.27)) (justify left bottom))
+    )
+    (property "Sheetfile" "power.kicad_sch" (at 67.31 27.2546 0)
+      (effects (font (size 1.27 1.27)) (justify left top))
+    )
+    (pin "Foo" input (at 67.31 45.72 180)
+      (effects (font (size 1.27 1.27)) (justify right))
+    )
+    (instances
+      (project "microgame2"
+        (path "/ebfd9da1-8e1c-4303-a1cc-72875a794180" (page "7"))
+      )
+    )
+  )
+  (sheet (at 67.31 53.8984 0) (size 40.64 6.35) (fields_autoplaced)
+    (stroke (width 0) (type solid))
+    (fill (color 0 0 0 0.0000))
+    (property "Sheetname" "Power4" (at 67.31 19.6084 0)
+      (effects (font (size 1.27 1.27)) (justify left bottom))
+    )
+    (property "Sheetfile" "power.kicad_sch" (at 67.31 27.2546 0)
+      (effects (font (size 1.27 1.27)) (justify left top))
+    )
+    (pin "Foo" input (at 92.71 60.96 270)
+      (effects (font (size 1.27 1.27)) (justify right))
+    )
+    (instances
+      (project "microgame2"
+        (path "/ebfd9da1-8e1c-4303-a1cc-72875a794180" (page "7"))
+      )
     )
   )
